File: hw/FTDI.sch (KiCad schematic (older format))
At the start: 0 parts

Commit message: Project divided in parts - MAX10board:                                -> FTDI 	                       -> POWER
 On branch PowerSchematic
 Changes to be committed:
	copied:     hw/max10.sch -> hw/FTDI.sch
	modified:   hw/max10-cache.lib
	deleted:    hw/max10.bak
	modified:   hw/max10.sch
 Untracked files:
	hw/FTDI.pro
Parts:
- added C? (x2): C, symbol C
- added CON?: BARREL_JACK, symbol BARREL_JACK
- added P?: USB_A, symbol USB_A
- added U?: FT2232H, symbol FT2232H
- added X?: CRYSTAL_SMD, symbol CRYSTAL_SMD
Connections:
- new net: P?.2 (D-), U?.7 (DM)
- new net: P?.3 (D+), U?.8 (DP)
- new net: C?.1, U?.2 (OSCI), X?.1
- new net: C?.1, U?.3 (OSCO), X?.2
- new net +1V8: U?.12 (VCORE), U?.37 (VCORE), U?.64 (VCORE)
- new net +3V3: U?.20 (VCCIO), U?.31 (VCCIO), U?.42 (VCCIO), U?.56 (VCCIO)
- new net GND: C?.2, C?.2, P?.4 (GND), U?.1 (GND), U?.10 (AGND), U?.11 (GND), U?.13 (TEST), U?.15 (GND), U?.25 (GND), U?.35 (GND), U?.47 (GND), U?.5 (GND), U?.51 (GND)
