File: hw/max10.sch (KiCad schematic (older format))
At the start: 6 parts

Commit message: Project divided in parts - MAX10board:                                -> FTDI 	                       -> POWER
 On branch PowerSchematic
 Changes to be committed:
	copied:     hw/max10.sch -> hw/FTDI.sch
	modified:   hw/max10-cache.lib
	deleted:    hw/max10.bak
	modified:   hw/max10.sch
 Untracked files:
	hw/FTDI.pro
Parts:
- removed C? (x2): C, symbol C
- removed CON?: BARREL_JACK, symbol BARREL_JACK
- removed P?: USB_A, symbol USB_A
- removed U?: FT2232H, symbol FT2232H
- removed X?: CRYSTAL_SMD, symbol CRYSTAL_SMD
